File: Schemat ideowy/new/Bartosz.Nowakowski.sch (EAGLE design)
At the start: 21 parts, among them J2 6_PIN_SERIAL_CABLEPTH, U1 ESP8266, U2 4MB Flash, Y1 CRYSTAL-26MHZSMD-3.2X2.5

Commit message: update
Parts:
- added JP1: 1, jumper:JP1E
- R8: value 12k -> 1k; device SparkFun-Resistors:12KOHM-0603-1/10W-1% -> SparkFun-Resistors:1KOHM-0603-1/10W-1%
Connections:
- new net GPIO0: JP1.2, R8.1, U1.SPICS2/GPIO0
- new net GPIO2: R7.1, U1.GPIO2
- new net N$10: J2.1, JP1.1
- new net U0RXI: J2.3, U1.U0RXD
- new net U0TXO: J2.2, U1.U0TXD
- net +3V3: now also J2.4
- net GND: now also J2.6
Other:
- moved on the sheet: C6, R2, R6, R7, R8, S1
